Commit message: Imported upstream version '0.1.6' of 'upstream'

File: urdf/sick_lms1xx.urdf.xacro (robot description, xacro)
@@ -26,5 +26,6 @@
 -->
 <robot xmlns:xacro="http://ros.org/wiki/xacro">
-  <xacro:macro name="sick_lms1xx" params="frame:=laser topic:=scan" >
+  <xacro:macro name="sick_lms1xx" params="frame:=laser topic:=scan sample_size:=720 update_rate:=50
+               min_angle:=-2.35619 max_angle:=2.35619 min_range:=0.1 max_range:=30.0 robot_namespace:=/" >
     <link name="${frame}">
       <inertial>
@@ -54,17 +55,17 @@
         <pose>0 0 0 0 0 0</pose>
         <visualize>false</visualize>
-        <update_rate>50</update_rate>
+        <update_rate>${update_rate}</update_rate>
         <ray>
           <scan>
             <horizontal>
-              <samples>720</samples>
+              <samples>${sample_size}</samples>
               <resolution>1</resolution>
-              <min_angle>-2.35619</min_angle>
-              <max_angle>2.35619</max_angle>
+              <min_angle>${min_angle}</min_angle>
+              <max_angle>${max_angle}</max_angle>
             </horizontal>
           </scan>
           <range>
-            <min>0.10</min>
-            <max>30.0</max>
+            <min>${min_range}</min>
+            <max>${max_range}</max>
             <resolution>0.01</resolution>
           </range>
@@ -78,4 +79,5 @@
           <topicName>${topic}</topicName>
           <frameName>${frame}</frameName>
+          <robotNamespace>${robot_namespace}</robotNamespace>
         </plugin>
       </sensor>

Commit message: Imported upstream version '1.0.0' of 'upstream'

File: urdf/sick_lms1xx.urdf.xacro (robot description, xacro)
@@ -40,5 +40,5 @@
         <geometry>
           <!-- Origin of this mesh is the focal point of the LIDAR. -->
-          <mesh filename="package://lms1xx/meshes/sick-lms1xx.dae" />
+          <mesh filename="file://$(find lms1xx)/meshes/sick-lms1xx.dae" />
         </geometry>
       </visual>
@@ -76,8 +76,18 @@
           </noise>
         </ray>
-        <plugin name="gazebo_ros_laser" filename="libgazebo_ros_laser.so">
-          <topicName>${topic}</topicName>
-          <frameName>${frame}</frameName>
-          <robotNamespace>${robot_namespace}</robotNamespace>
+        <plugin name="${frame}_scan" filename="libgazebo_ros_ray_sensor.so">
+          <ros>
+            <remapping>~/out:=${topic}</remapping>
+            <qos>
+              <topic name="${topic}">
+                  <publisher>
+                      <reliability>best_effort</reliability>
+                  </publisher>
+              </topic>
+            </qos>
+          </ros>
+          <frame_name>${frame}</frame_name>
+          <robot_namespace>${robot_namespace}</robot_namespace>
+          <output_type>sensor_msgs/LaserScan</output_type>
         </plugin>
       </sensor>
